File: kana60-acrylic-plates.kicad_pcb (KiCad board)
At the start: 2 copper layers, 285.4 x 115.5 mm, 9 parts

Commit message: update acrylic plates
Parts:
- added REF10: MountingHole_2.2mm_M2_Pad, MountingHole:MountingHole_2.2mm_M2_Pad, F.Cu at (19.7, 144.6)
- added REF11: MountingHole_2.2mm_M2_Pad, MountingHole:MountingHole_2.2mm_M2_Pad, F.Cu at (253.2, 144.6)
- added REF12: MountingHole_2.2mm_M2_Pad, MountingHole:MountingHole_2.2mm_M2_Pad, F.Cu at (19.7, 157.3)
- added REF13: MountingHole_2.2mm_M2_Pad, MountingHole:MountingHole_2.2mm_M2_Pad, F.Cu at (253.2, 157.3)
Other:
- board size 285.4 x 115.5 mm -> 285.4 x 141.9 mm

Commit message: update Edge.Cuts
Parts:
- moved REF10 2.41 mm to (19.8, 142.2)
- moved REF11 2.41 mm to (253.3, 142.2)
- moved REF12 2.41 mm to (19.8, 154.9)
- moved REF13 2.41 mm to (253.3, 154.9)
Other:
- board size 285.4 x 141.9 mm -> 285.6 x 139.6 mm

Commit message: update acrylic plates
Parts:
- moved REF10 0.13 mm to (19.7, 142.2)
- moved REF12 0.13 mm to (19.7, 154.9)
- moved REF11 0.13 mm to (253.2, 142.2)
- moved REF13 0.13 mm to (253.2, 154.9)
Other:
- board size 285.6 x 139.6 mm -> 285.5 x 139.6 mm
Changed lines of the file:
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@@
   )
   (module MountingHole:MountingHole_2.2mm_M2_Pad (layer F.Cu)
-    (at 253.330988 142.2267)
+    (at 253.200988 142.2267)
     (descr "Mounting Hole 2.2mm, M2")
     (tags "mounting hole 2.2mm m2")
@@
   )
   (module MountingHole:MountingHole_2.2mm_M2_Pad (layer F.Cu)
-    (at 19.835988 154.9267)
+    (at 19.705988 154.9267)
     (descr "Mounting Hole 2.2mm, M2")
     (tags "mounting hole 2.2mm m2")
@@
   )
   (module MountingHole:MountingHole_2.2mm_M2_Pad (layer F.Cu)
-    (at 19.835988 142.2267)
+    (at 19.705988 142.2267)
     (descr "Mounting Hole 2.2mm, M2")
     (tags "mounting hole 2.2mm m2")
@@
   )
   (module MountingHole:MountingHole_2.2mm_M2_Pad (layer F.Cu)
-    (at 253.330988 154.9267)
+    (at 253.200988 154.9267)
     (descr "Mounting Hole 2.2mm, M2")
     (tags "mounting hole 2.2mm m2")
@@
     (pad 1 thru_hole circle (at 0 0) (size 4.4 4.4) (drill 2.2) (layers *.Cu *.Mask))
   )
-  (gr_line (start 16.152988 140.0677) (end 16.152988 157.0857) (layer Edge.Cuts) (width 0.2))
-  (gr_line (start 301.648988 140.0677) (end 301.648988 157.0857) (layer Edge.Cuts) (width 0.2))
-  (gr_circle (center 19.835988 142.2267) (end 20.935988 142.2267) (layer Edge.Cuts) (width 0.2))
-  (gr_circle (center 19.835988 154.9267) (end 20.935988 154.9267) (layer Edge.Cuts) (width 0.2))
-  (gr_circle (center 253.330988 154.9267) (end 254.430988 154.9267) (layer Edge.Cuts) (width 0.2))
-  (gr_circle (center 253.330988 142.2267) (end 254.430988 142.2267) (layer Edge.Cuts) (width 0.2))
-  (gr_line (start 17.930988 138.2897) (end 299.870988 138.2897) (layer Edge.Cuts) (width 0.2))
-  (gr_arc (start 17.930988 140.0677) (end 17.930988 138.2897) (angle -90) (layer Edge.Cuts) (width 0.2))
-  (gr_arc (start 299.870988 140.0677) (end 301.648988 140.0677) (angle -90) (layer Edge.Cuts) (width 0.2))
-  (gr_line (start 299.870988 158.8637) (end 17.930988 158.8637) (layer Edge.Cuts) (width 0.2))
-  (gr_line (start 299.870988 157.0857) (end 301.648988 158.8637) (layer Dwgs.User) (width 0.15))
-  (gr_arc (start 299.870988 157.0857) (end 299.870988 158.8637) (angle -90) (layer Edge.Cuts) (width 0.2))
-  (gr_line (start 16.152988 158.8637) (end 17.930988 157.0857) (layer Dwgs.User) (width 0.15))
-  (gr_arc (start 17.930988 157.0857) (end 16.152988 157.0857) (angle -90) (layer Edge.Cuts) (width 0.2))
-  (gr_line (start 16.152988 158.8637) (end 17.930988 160.6417) (layer Dwgs.User) (width 0.15))
-  (gr_arc (start 17.930988 160.6417) (end 17.930988 158.8637) (angle -90) (layer Dwgs.User) (width 0.15))
-  (gr_line (start 299.870988 160.6417) (end 301.648988 158.8637) (layer Dwgs.User) (width 0.15))
-  (gr_arc (start 299.870988 160.6417) (end 301.648988 160.6417) (angle -90) (layer Dwgs.User) (width 0.15))
+  (gr_line (start 16.022988 140.0677) (end 16.022988 157.0857) (layer Edge.Cuts) (width 0.2))
+  (gr_line (start 301.518988 140.0677) (end 301.518988 157.0857) (layer Edge.Cuts) (width 0.2))
+  (gr_circle (center 19.705988 142.2267) (end 20.805988 142.2267) (layer Edge.Cuts) (width 0.2))
+  (gr_circle (center 19.705988 154.9267) (end 20.805988 154.9267) (layer Edge.Cuts) (width 0.2))
+  (gr_circle (center 253.200988 154.9267) (end 254.300988 154.9267) (layer Edge.Cuts) (width 0.2))
+  (gr_circle (center 253.200988 142.2267) (end 254.300988 142.2267) (layer Edge.Cuts) (width 0.2))
+  (gr_line (start 17.800988 138.2897) (end 299.740988 138.2897) (layer Edge.Cuts) (width 0.2))
+  (gr_arc (start 17.800988 140.0677) (end 17.800988 138.2897) (angle -90) (layer Edge.Cuts) (width 0.2))
+  (gr_arc (start 299.740988 140.0677) (end 301.518988 140.0677) (angle -90) (layer Edge.Cuts) (width 0.2))
+  (gr_line (start 299.740988 158.8637) (end 17.800988 158.8637) (layer Edge.Cuts) (width 0.2))
+  (gr_line (start 299.740988 157.0857) (end 301.518988 158.8637) (layer Cmts.User) (width 0.15))
+  (gr_arc (start 299.740988 157.0857) (end 299.740988 158.8637) (angle -90) (layer Edge.Cuts) (width 0.2))
+  (gr_line (start 16.022988 158.8637) (end 17.800988 157.0857) (layer Cmts.User) (width 0.15))
+  (gr_arc (start 17.800988 157.0857) (end 16.022988 157.0857) (angle -90) (layer Edge.Cuts) (width 0.2))
+  (gr_line (start 16.022988 158.8637) (end 17.800988 160.6417) (layer Cmts.User) (width 0.15))
+  (gr_arc (start 17.800988 160.6417) (end 17.800988 158.8637) (angle -90) (layer Cmts.User) (width 0.15))
+  (gr_line (start 299.740988 160.6417) (end 301.518988 158.8637) (layer Cmts.User) (width 0.15))
+  (gr_arc (start 299.740988 160.6417) (end 301.518988 160.6417) (angle -90) (layer Cmts.User) (width 0.15))
   (gr_circle (center 224.559988 125.4627) (end 225.659988 125.4627) (layer Edge.Cuts) (width 0.2))
   (gr_circle (center 63.523988 125.4627) (end 64.623988 125.4627) (layer Edge.Cuts) (width 0.2))
@@
   (gr_circle (center 19.708988 35.9277) (end 20.808988 35.9277) (layer Edge.Cuts) (width 0.2))
   (gr_circle (center 19.708988 23.2277) (end 20.808988 23.2277) (layer Edge.Cuts) (width 0.2))
-  (gr_arc (start 299.743988 41.6427) (end 301.521988 41.6427) (angle -90) (layer Dwgs.User) (width 0.15))
-  (gr_line (start 299.743988 41.6427) (end 301.521988 39.8647) (layer Dwgs.User) (width 0.15))
-  (gr_arc (start 17.803988 41.6427) (end 17.803988 39.8647) (angle -90) (layer Dwgs.User) (width 0.15))
-  (gr_line (start 16.025988 39.8647) (end 17.803988 41.6427) (layer Dwgs.User) (width 0.15))
-  (gr_arc (start 17.803988 38.0867) (end 16.025988 38.0867) (angle -90) (layer Dwgs.User) (width 0.15))
-  (gr_line (start 16.025988 39.8647) (end 17.803988 38.0867) (layer Dwgs.User) (width 0.15))
-  (gr_arc (start 299.743988 38.0867) (end 299.743988 39.8647) (angle -90) (layer Dwgs.User) (width 0.15))
-  (gr_line (start 299.743988 38.0867) (end 301.521988 39.8647) (layer Dwgs.User) (width 0.15))
-  (gr_line (start 304.823988 39.8647) (end 12.723988 39.8647) (layer Dwgs.User) (width 0.15))
+  (gr_arc (start 299.743988 41.6427) (end 301.521988 41.6427) (angle -90) (layer Cmts.User) (width 0.15))
+  (gr_line (start 299.743988 41.6427) (end 301.521988 39.8647) (layer Cmts.User) (width 0.15))
+  (gr_arc (start 17.803988 41.6427) (end 17.803988 39.8647) (angle -90) (layer Cmts.User) (width 0.15))
+  (gr_line (start 16.025988 39.8647) (end 17.803988 41.6427) (layer Cmts.User) (width 0.15))
+  (gr_arc (start 17.803988 38.0867) (end 16.025988 38.0867) (angle -90) (layer Cmts.User) (width 0.15))
+  (gr_line (start 16.025988 39.8647) (end 17.803988 38.0867) (layer Cmts.User) (width 0.15))
+  (gr_arc (start 299.743988 38.0867) (end 299.743988 39.8647) (angle -90) (layer Cmts.User) (width 0.15))
+  (gr_line (start 299.743988 38.0867) (end 301.521988 39.8647) (layer Cmts.User) (width 0.15))
+  (gr_line (start 304.823988 39.8647) (end 12.723988 39.8647) (layer Cmts.User) (width 0.15))
   (gr_arc (start 299.743988 21.0687) (end 301.521988 21.0687) (angle -90) (layer Edge.Cuts) (width 0.2))
   (gr_arc (start 17.803988 21.0687) (end 17.803988 19.2907) (angle -90) (layer Edge.Cuts) (width 0.2))

Commit message: update dimention lines
Other:
- board text added: "4-φ2.2"
- board text added: "9-φ2.2"

Commit message: move lines into frame
Parts:
- moved REF8 36.1 mm to (93.5, 145.5)
- moved REF9 36.1 mm to (254.6, 145.5)
- moved REF1 36.1 mm to (49.7, 43.2)
- moved REF10 36.1 mm to (49.7, 162.2)
- moved REF11 36.1 mm to (283.2, 162.2)
- moved REF12 36.1 mm to (49.7, 174.9)
- moved REF13 36.1 mm to (283.2, 174.9)
- moved REF3 36.1 mm to (49.7, 55.9)
- moved REF5 36.1 mm to (71.5, 88.1)
- moved REF6 36.1 mm to (306.3, 88.1)
- moved REF7 36.1 mm to (174.3, 107.4)
- moved REF2 36.1 mm to (283.2, 43.2)
- moved REF4 36.1 mm to (283.2, 55.9)
