File: kana60-top-plate.kicad_pcb (KiCad board)
At the start: 2 copper layers, 285.4 x 115.5 mm, 13 parts, among them SW29 SW_PUSH, SW42 SW_PUSH, SW43 SW_PUSH, SW60 SW_PUSH, SW61 SW_PUSH, SW68 SW_PUSH, SW69 SW_PUSH, SW70 SW_PUSH

Commit message: update top plate
Parts:
- removed SW29: SW_PUSH, Keebio-Parts:Hybrid_PCB_175H
- removed SW42, SW43, SW60, SW70: SW_PUSH, Keebio-Parts:Hybrid_PCB_200H
- removed SW61, SW68, SW69: SW_PUSH, Keebio-Parts:Hybrid_PCB_100H
Other:
- board size 285.4 x 115.5 mm -> 285.4 x 94.9 mm

Commit message: update Edge.Cuts
Other:
- board size 285.4 x 94.9 mm -> 285.5 x 95 mm

Commit message: add plane to top plate
Routing:
- added copper zone on B.Cu, net (none)
- added copper zone on F.Cu, net (none)
Changed lines of the file:
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@@
   (gr_line (start 16.025988 133.0827) (end 16.025988 41.6427) (layer Edge.Cuts) (width 0.2))
   (gr_line (start 301.521988 133.0827) (end 301.521988 41.6427) (layer Edge.Cuts) (width 0.2))
+  (zone (net 0) (net_name "") (layer F.Cu) (hatch edge 0.508)
+    (connect_pads (clearance 0.508))
+    (min_thickness 0.254)
+    (fill yes (arc_segments 32) (thermal_gap 0.508) (thermal_bridge_width 0.508))
+    (polygon
+      (pts
+        (xy 16.025988 39.8647) (xy 301.521988 39.8647) (xy 301.521988 134.8607) (xy 16.025988 134.8607)
+      )
+    )
+  )
+  (zone (net 0) (net_name "") (layer B.Cu) (hatch edge 0.508)
+    (connect_pads (clearance 0.508))
+    (min_thickness 0.254)
+    (fill yes (arc_segments 32) (thermal_gap 0.508) (thermal_bridge_width 0.508))
+    (polygon
+      (pts
+        (xy 16.025988 39.8647) (xy 301.521988 39.8647) (xy 301.521988 134.8607) (xy 16.025988 134.8607)
+      )
+    )
+  )
 )

Commit message: fix stabilizer interfere
Other:
- outline, holes or cut-outs redrawn
Changed lines of the file:
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@@
   (gr_line (start 172.33675 119.02655) (end 172.33675 119.94705) (layer Edge.Cuts) (width 0.2))
   (gr_line (start 172.33675 119.94705) (end 174.06145 119.94705) (layer Edge.Cuts) (width 0.2))
-  (gr_line (start 174.06145 119.94705) (end 174.06145 123.17725) (layer Edge.Cuts) (width 0.2))
-  (gr_line (start 174.06145 123.17725) (end 174.88695 123.17725) (layer Edge.Cuts) (width 0.2))
+  (gr_line (start 174.88695 119.94705) (end 174.88695 123.17725) (layer Edge.Cuts) (width 0.2))
+  (gr_line (start 174.06145 119.94705) (end 174.88695 119.94705) (layer Edge.Cuts) (width 0.2))
   (gr_line (start 174.88695 123.17725) (end 174.88695 125.97597) (layer Edge.Cuts) (width 0.2))
-  (gr_line (start 174.88695 125.97597) (end 174.06145 125.97597) (layer Edge.Cuts) (width 0.2))
-  (gr_line (start 174.06145 125.97597) (end 174.06145 132.24606) (layer Edge.Cuts) (width 0.2))
+  (gr_line (start 174.88695 132.24606) (end 174.06145 132.24606) (layer Edge.Cuts) (width 0.2))
+  (gr_line (start 174.88695 125.97597) (end 174.88695 132.24606) (layer Edge.Cuts) (width 0.2))
   (gr_line (start 174.06145 132.24606) (end 172.33675 132.24606) (layer Edge.Cuts) (width 0.2))
   (gr_line (start 172.33675 132.24606) (end 172.33675 133.22723) (layer Edge.Cuts) (width 0.2))
@@
   (gr_line (start 118.44975 133.22723) (end 118.44975 132.4762) (layer Edge.Cuts) (width 0.2))
   (gr_line (start 292.03375 61.75115) (end 289.23375 61.75115) (layer Edge.Cuts) (width 0.2))
-  (gr_line (start 292.03375 62.57665) (end 292.03375 61.75115) (layer Edge.Cuts) (width 0.2))
-  (gr_line (start 295.26375 62.57665) (end 292.03375 62.57665) (layer Edge.Cuts) (width 0.2))
+  (gr_line (start 295.26375 62.57665) (end 295.26375 61.75115) (layer Edge.Cuts) (width 0.2))
+  (gr_line (start 295.26375 61.75115) (end 292.03375 61.75115) (layer Edge.Cuts) (width 0.2))
   (gr_line (start 295.26375 64.30205) (end 295.26375 62.57665) (layer Edge.Cuts) (width 0.2))
   (gr_line (start 296.18475 64.30205) (end 295.26375 64.30205) (layer Edge.Cuts) (width 0.2))
@@
   (gr_line (start 282.96475 64.30205) (end 281.98375 64.30205) (layer Edge.Cuts) (width 0.2))
   (gr_line (start 282.96475 62.57665) (end 282.96475 64.30205) (layer Edge.Cuts) (width 0.2))
-  (gr_line (start 289.23375 62.57665) (end 282.96475 62.57665) (layer Edge.Cuts) (width 0.2))
-  (gr_line (start 289.23375 61.75115) (end 289.23375 62.57665) (layer Edge.Cuts) (width 0.2))
+  (gr_line (start 289.23375 61.75115) (end 282.96475 61.75115) (layer Edge.Cuts) (width 0.2))
+  (gr_line (start 282.96475 61.75115) (end 282.96475 62.57665) (layer Edge.Cuts) (width 0.2))
   (gr_line (start 294.62375 70.85175) (end 294.62375 69.326351) (layer Edge.Cuts) (width 0.2))
   (gr_line (start 283.92375 69.326351) (end 283.92375 70.85175) (layer Edge.Cuts) (width 0.2))
@@
   (gr_line (start 295.26375 91.40245) (end 296.18475 91.40245) (layer Edge.Cuts) (width 0.2))
   (gr_line (start 295.26375 93.12755) (end 295.26375 91.40245) (layer Edge.Cuts) (width 0.2))
-  (gr_line (start 292.03375 93.12755) (end 295.26375 93.12755) (layer Edge.Cuts) (width 0.2))
-  (gr_line (start 292.03375 93.95165) (end 292.03375 93.12755) (layer Edge.Cuts) (width 0.2))
+  (gr_line (start 292.03375 93.95165) (end 295.26375 93.95165) (layer Edge.Cuts) (width 0.2))
+  (gr_line (start 295.26375 93.95165) (end 295.26375 93.12755) (layer Edge.Cuts) (width 0.2))
   (gr_line (start 289.23375 93.95165) (end 292.03375 93.95165) (layer Edge.Cuts) (width 0.2))
-  (gr_line (start 289.23375 93.12755) (end 289.23375 93.95165) (layer Edge.Cuts) (width 0.2))
-  (gr_line (start 282.96475 93.12755) (end 289.23375 93.12755) (layer Edge.Cuts) (width 0.2))
+  (gr_line (start 282.96475 93.12755) (end 282.96475 93.95165) (layer Edge.Cuts) (width 0.2))
+  (gr_line (start 282.96475 93.95165) (end 289.23375 93.95165) (layer Edge.Cuts) (width 0.2))
   (gr_line (start 282.96475 91.40245) (end 282.96475 93.12755) (layer Edge.Cuts) (width 0.2))
   (gr_line (start 281.98375 91.40245) (end 282.96475 91.40245) (layer Edge.Cuts) (width 0.2))
@@
   (gr_line (start 50.87155 100.89705) (end 50.87155 99.97655) (layer Edge.Cuts) (width 0.2))
   (gr_line (start 52.59675 100.89705) (end 50.87155 100.89705) (layer Edge.Cuts) (width 0.2))
-  (gr_line (start 52.59675 104.12725) (end 52.59675 100.89705) (layer Edge.Cuts) (width 0.2))
-  (gr_line (start 53.42225 104.12725) (end 52.59675 104.12725) (layer Edge.Cuts) (width 0.2))
+  (gr_line (start 53.42225 104.12725) (end 53.42225 100.89705) (layer Edge.Cuts) (width 0.2))
+  (gr_line (start 53.42225 100.89705) (end 52.59675 100.89705) (layer Edge.Cuts) (width 0.2))
   (gr_line (start 53.42225 106.92595) (end 53.42225 104.12725) (layer Edge.Cuts) (width 0.2))
-  (gr_line (start 52.59675 106.92595) (end 53.42225 106.92595) (layer Edge.Cuts) (width 0.2))
-  (gr_line (start 52.59675 113.19605) (end 52.59675 106.92595) (layer Edge.Cuts) (width 0.2))
+  (gr_line (start 52.59675 113.19605) (end 53.42225 113.19605) (layer Edge.Cuts) (width 0.2))
+  (gr_line (start 53.42225 113.19605) (end 53.42225 106.92595) (layer Edge.Cuts) (width 0.2))
   (gr_line (start 50.87155 113.19605) (end 52.59675 113.19605) (layer Edge.Cuts) (width 0.2))
   (gr_line (start 50.87155 114.17725) (end 50.87155 113.19605) (layer Edge.Cuts) (width 0.2))
@@
   (gr_line (start 23.77241 113.19605) (end 23.77241 114.17725) (layer Edge.Cuts) (width 0.2))
   (gr_line (start 22.04712 113.19605) (end 23.77241 113.19605) (layer Edge.Cuts) (width 0.2))
-  (gr_line (start 22.04712 106.92595) (end 22.04712 113.19605) (layer Edge.Cuts) (width 0.2))
-  (gr_line (start 21.22169 106.92595) (end 22.04712 106.92595) (layer Edge.Cuts) (width 0.2))
+  (gr_line (start 21.22169 106.92595) (end 21.22169 113.19605) (layer Edge.Cuts) (width 0.2))
+  (gr_line (start 21.22169 113.19605) (end 22.04712 113.19605) (layer Edge.Cuts) (width 0.2))
   (gr_line (start 21.22169 104.12725) (end 21.22169 106.92595) (layer Edge.Cuts) (width 0.2))
-  (gr_line (start 22.04712 104.12725) (end 21.22169 104.12725) (layer Edge.Cuts) (width 0.2))
-  (gr_line (start 22.04712 100.89705) (end 22.04712 104.12725) (layer Edge.Cuts) (width 0.2))
+  (gr_line (start 22.04712 100.89705) (end 21.22169 100.89705) (layer Edge.Cuts) (width 0.2))
+  (gr_line (start 21.22169 100.89705) (end 21.22169 104.12725) (layer Edge.Cuts) (width 0.2))
   (gr_line (start 23.77241 100.89705) (end 22.04712 100.89705) (layer Edge.Cuts) (width 0.2))
   (gr_line (start 23.77241 99.97655) (end 23.77241 100.89705) (layer Edge.Cuts) (width 0.2))
@@
   (gr_line (start 116.64075 132.24606) (end 116.64075 133.22723) (layer Edge.Cuts) (width 0.2))
   (gr_line (start 114.91605 132.24606) (end 116.64075 132.24606) (layer Edge.Cuts) (width 0.2))
-  (gr_line (start 114.91605 125.97597) (end 114.91605 132.24606) (layer Edge.Cuts) (width 0.2))
-  (gr_line (start 114.09055 125.97597) (end 114.91605 125.97597) (layer Edge.Cuts) (width 0.2))
+  (gr_line (start 114.09055 125.97597) (end 114.09055 132.24606) (layer Edge.Cuts) (width 0.2))
+  (gr_line (start 114.09055 132.24606) (end 114.91605 132.24606) (layer Edge.Cuts) (width 0.2))
   (gr_line (start 114.09055 123.17725) (end 114.09055 125.97597) (layer Edge.Cuts) (width 0.2))
-  (gr_line (start 114.91605 123.17725) (end 114.09055 123.17725) (layer Edge.Cuts) (width 0.2))
-  (gr_line (start 114.91605 119.94705) (end 114.91605 123.17725) (layer Edge.Cuts) (width 0.2))
+  (gr_line (start 114.91605 119.94705) (end 114.09055 119.94705) (layer Edge.Cuts) (width 0.2))
+  (gr_line (start 114.09055 119.94705) (end 114.09055 123.17725) (layer Edge.Cuts) (width 0.2))
   (gr_line (start 116.64075 119.94705) (end 114.91605 119.94705) (layer Edge.Cuts) (width 0.2))
   (gr_line (start 116.64075 119.02655) (end 116.64075 119.94705) (layer Edge.Cuts) (width 0.2))
